File: EcoMecPCB/EcoMecPCB.kicad_sch (KiCad schematic)
At the start: 28 parts, among them J2 LCpower, J3 Conn_01x02_Pin, J4 Conn_01x02_Pin, J5 Conn_01x03_Pin, J6 Conn_01x02_Pin, J7 Conn_01x03_Pin, J8 LCsignal, U1 CS1237-SO, U2 MT2492, U3 SIT65HVD230DR, U4 AZ1117-3.3, U6 STM32F_dev

Commit message: Pin layout done
Pin layout done
Connections:
- net DOUT: now also U6.15 (B7); no longer U6.35 (A1)
- net SCLK: now also U6.14 (B6); no longer U6.36 (A0)
- net UART_RX: now also U6.33 (A3); no longer U6.15 (B7)
- net UART_TX: now also U6.34 (A2); no longer U6.14 (B6)
Changed lines of the file:
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@@
-	)
-	(no_connect
-		(at 62.23 106.68)
 	)
 	(no_connect
@@
 	)
 	(no_connect
+		(at 62.23 114.3)
+	)
+	(no_connect
 		(at 62.23 83.82)
 	)
@@
 	)
 	(no_connect
-		(at 62.23 102.87)
+		(at 62.23 110.49)
 	)
 	(no_connect
@@
 	(wire
 		(pts
-			(xy 25.4 110.49) (xy 26.67 110.49)
-		)
-		(stroke
-			(width 0)
-			(type default)
-		)
-	)
-	(wire
-		(pts
 			(xy 62.23 60.96) (xy 63.5 60.96)
 		)
@@
 	(wire
 		(pts
+			(xy 17.78 110.49) (xy 26.67 110.49)
+		)
+		(stroke
+			(width 0)
+			(type default)
+		)
+	)
+	(wire
+		(pts
 			(xy 252.73 48.26) (xy 252.73 50.8)
 		)
@@
 	(wire
 		(pts
-			(xy 25.4 106.68) (xy 26.67 106.68)
-		)
-		(stroke
-			(width 0)
-			(type default)
-		)
-	)
-	(wire
-		(pts
 			(xy 189.23 68.58) (xy 189.23 66.04)
 		)
@@
 	(wire
 		(pts
+			(xy 62.23 106.68) (xy 72.39 106.68)
+		)
+		(stroke
+			(width 0)
+			(type default)
+		)
+	)
+	(wire
+		(pts
 			(xy 190.5 71.12) (xy 190.5 68.58)
 		)
@@
 	(wire
 		(pts
+			(xy 17.78 106.68) (xy 26.67 106.68)
+		)
+		(stroke
+			(width 0)
+			(type default)
+		)
+	)
+	(wire
+		(pts
 			(xy 82.55 69.85) (xy 82.55 73.66)
 		)
@@
 	(wire
 		(pts
-			(xy 62.23 110.49) (xy 66.04 110.49)
-		)
-		(stroke
-			(width 0)
-			(type default)
-		)
-	)
-	(wire
-		(pts
 			(xy 54.61 182.88) (xy 54.61 189.23)
 		)
@@
 	(wire
 		(pts
-			(xy 62.23 114.3) (xy 66.04 114.3)
-		)
-		(stroke
-			(width 0)
-			(type default)
-		)
-	)
-	(wire
-		(pts
 			(xy 93.98 152.4) (xy 93.98 162.56)
 		)
@@
 		(pts
 			(xy 31.75 171.45) (xy 31.75 173.99)
+		)
+		(stroke
+			(width 0)
+			(type default)
+		)
+	)
+	(wire
+		(pts
+			(xy 62.23 102.87) (xy 72.39 102.87)
 		)
 		(stroke
@@
 	)
 	(label "UART_RX"
-		(at 25.4 110.49 180)
+		(at 72.39 102.87 180)
 		(effects
 			(font
@@
 	)
 	(label "DOUT"
-		(at 66.04 110.49 0)
+		(at 17.78 110.49 0)
 		(effects
 			(font
@@
 	)
 	(label "UART_TX"
-		(at 25.4 106.68 180)
+		(at 72.39 106.68 180)
 		(effects
 			(font
@@
 	)
 	(label "SCLK"
-		(at 66.04 114.3 0)
-		(effects
-			(font
+		(at 17.78 106.68 0)
+		(effects
+			(font

Commit message: Schematic done
Schematic done
Parts:
- added J1: encoderPower, symbol Connector:Screw_Terminal_01x03
- added J9: encoderChannels, symbol Connector:Screw_Terminal_01x02
- added R6, R7: R, symbol Device:R
Connections:
- net +3.3V: now also R6.1, R7.1
- net +5V: now also J1.1 (Pin_1)
- net GND: now also J1.2 (Pin_2), J1.3 (Pin_3)
- net EncoderCH_A: now reaches U6.11 (B3)
- net EncoderCH_A: now also J9.1 (Pin_1), R6.2
- net EncoderCH_B: now reaches U6.12 (B4)
- net EncoderCH_B: now also J9.2 (Pin_2), R7.2
- no-connect marks 31 -> 29

Commit message: Schematic done
Schematic done
Parts:
- removed C8: 10u, symbol Device:C_Polarized
- added J10: MPU-6050, symbol Connector:Conn_01x08_Pin
- C2: value 100n -> 10u
- R6, R7: value R -> 4.7k
Connections:
- net +5V: now also J10.1 (Pin_1)
- net DOUT: now also U6.27 (B1); no longer U6.15 (B7)
- net GND: now also J10.2 (Pin_2)
- net SCLK: no longer U6.14 (B6)
- net MPU_INT: now reaches U6.25 (B11)
- net MPU_INT: now also J10.8 (Pin_8)
- net CS_CLK: now reaches U6.28 (B0)
- new net MPU_SCL: J10.3 (Pin_3), U6.14 (B6)
- new net MPU_SDA: J10.4 (Pin_4), U6.15 (B7)
Other:
- moved on the sheet: C2, J2

Commit message: Schematic inshallah Done
Schematic inshallah Done
Parts:
- removed J1: encoderPower, symbol Connector:Screw_Terminal_01x03
- removed J2: LCpower, symbol Connector:Screw_Terminal_01x02
- removed J8: LCsignal, symbol Connector:Screw_Terminal_01x02
- removed J9: encoderChannels, symbol Connector:Screw_Terminal_01x02
- added C10, C12, C8, C9: 100n, symbol Device:C
- added C11: 1u, symbol Device:C
- added J11: LC, symbol Connector:Screw_Terminal_01x04
- added J2: Encoder, symbol Connector:Screw_Terminal_01x05
- added R10, R11, R12, R8, R9: 1k, symbol Device:R
- added R13: 0, symbol Device:R
- added TP2: TestPoint, TestPoint:TestPoint_Pad_D1.5mm, symbol Connector:TestPoint
- added U5: TL431ACDBZR, EasyEDA:SOT-23-3_L3.0-W1.7-P0.95-LS2.9-BR, symbol EasyEDA:TL431ACDBZR
- C1: value 1u -> 100n
- C2: value 10u -> 100n
Connections:
- net +3.3V: now also R8.1
- net +5V: now also J2.1 (Pin_1)
- net CS_CLK: now also U6.11 (B3); no longer U6.28 (B0)
- net DOUT: now also U6.12 (B4); no longer U6.27 (B1)
- net EncoderCH_A: now also U6.27 (B1), C8.2, R9.1; no longer R6.2, U6.11 (B3)
- net EncoderCH_B: now also U6.28 (B0), C9.2, R10.1; no longer R7.2, U6.12 (B4)
- net GND: now also C11.1, C12.1, C8.1, C9.1, J11.2 (Pin_2), J2.2 (Pin_2), J2.3 (Pin_3), U5.1 (CATHODE)
- net S+: now also C10.1, R11.1
- net S-: now also C10.2, R12.1
- net VREF: now also C11.2, C12.2, J11.1 (Pin_1), R13.1, R8.2, TP2.1, U5.2 (REF), U5.3 (ANODE); no longer U1.8 (REFOUT)
- new net: R13.2, U1.8 (REFOUT)
- new net: J11.3 (Pin_3), R11.2
- new net: J11.4 (Pin_4), R12.2
- new net: J2.4 (Pin_4), R6.2, R9.2
- new net: J2.5 (Pin_5), R10.2, R7.2
Other:
- moved on the sheet: J10, J7, R6, R7

Commit message: Update
Parts:
- removed U5: TL431ACDBZR, EasyEDA:SOT-23-3_L3.0-W1.7-P0.95-LS2.9-BR, symbol EasyEDA:TL431ACDBZR
- added U7: TL431DBZ, Package_TO_SOT_SMD:SOT-23, symbol Reference_Voltage:TL431DBZ
- C1, C10, C11, C12, C2, C8, C9: footprint (none) -> Capacitor_SMD:C_1206_3216Metric_Pad1.33x1.80mm_HandSolder
- C3, C4, C5, C6, C7: footprint LED_SMD:LED_1206_3216Metric_Pad1.42x1.75mm_HandSolder -> Capacitor_SMD:C_1206_3216Metric_Pad1.33x1.80mm_HandSolder
- J10: footprint (none) -> Connector_PinHeader_2.54mm:PinHeader_1x08_P2.54mm_Vertical
- J11: footprint (none) -> TerminalBlock_Phoenix:TerminalBlock_Phoenix_PT-1,5-4-3.5-H_1x04_P3.50mm_Horizontal
- J2: footprint (none) -> TerminalBlock_Phoenix:TerminalBlock_Phoenix_PT-1,5-5-3.5-H_1x05_P3.50mm_Horizontal
- R10, R11, R12, R13, R6, R7, R8, R9: footprint (none) -> Resistor_SMD:R_1206_3216Metric_Pad1.30x1.75mm_HandSolder
Connections:
- net GND: now also U7.3 (A)
- net VREF: now also U7.1 (K), U7.2 (REF)
