File: EcoMecPCB/EcoMecPCB.kicad_pcb (KiCad board)
At the start: 2 copper layers, 47.5 x 97.7 mm, 43 parts, among them J10 MPU-6050, J11 LC, J2 Encoder, J3 Conn_01x02_Pin, J4 Conn_01x02_Pin, J5 Conn_01x03_Pin, J6 Conn_01x02_Pin, J7 Conn_01x03_Pin, U1 CS1237-SO, U2 MT2492, U3 SIT65HVD230DR, U4 AZ1117-3.3, U6 STM32F_dev, U7 TL431DBZ

Commit message: Finished routing and layout
finished layout
finished routing
Parts:
- moved J3 199.3 mm to (186.2, 141.0)
- moved C4 190.4 mm to (178.5, 139.0), turned to 180 degrees
- moved C6 188.6 mm to (183.0, 131.4), turned to -90 degrees
- moved C3 186.5 mm to (180.9, 124.5)
- moved R2 185.2 mm to (178.6, 136.0)
- moved J4 183.9 mm to (178.0, 142.5), turned to 90 degrees
- moved C7 179.3 mm to (180.9, 120.5), turned to 180 degrees
- moved U2 178.5 mm to (179.1, 131.3), turned to 180 degrees
- moved L1 177.3 mm to (188.5, 131.7), turned to 90 degrees
- moved R3 176.8 mm to (173.9, 130.5)
- moved R4 176.4 mm to (173.9, 133.0), turned to 180 degrees
- moved U4 173.2 mm to (187.5, 122.0), turned to 90 degrees
- moved TP1 172.3 mm to (190.5, 117.5)
- moved RV1 163.4 mm to (174.5, 119.4), turned to 90 degrees
- moved J7 132.8 mm to (189.0, 83.5), turned to -90 degrees
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Routing:
- net +5V: track 0.00 -> 145.6 mm, vias 0 -> 4
- net +3.3V: track 0.00 -> 133.6 mm, vias 0 -> 13
- net /EncoderCH_A: track 0.00 -> 96.7 mm, vias 0 -> 4
- net /EncoderCH_B: track 0.00 -> 88.8 mm, vias 0 -> 4
- net /MPU_INT: track 0.00 -> 69.2 mm, vias 0 -> 2
- net /MPU_SCL: track 0.00 -> 69.1 mm, vias 0 -> 4
- net /MPU_SDA: track 0.00 -> 65.3 mm, vias 0 -> 4
- net /UART_RX: track 0.00 -> 62.7 mm, vias 0 -> 4
- net /UART_TX: track 0.00 -> 62.4 mm, vias 0 -> 4
- net /VREF: track 0.00 -> 53.3 mm, vias 0 -> 2
- net /DOUT: track 0.00 -> 50.9 mm, vias 0 -> 4
- net /CAN_L: track 0.00 -> 17.7 mm, vias 0 -> 4
- net Net-(J4-Pin_1): track 0.00 -> 17.0 mm, vias 0 -> 4
- net /CAN_RXD: track 0.00 -> 14.0 mm, vias 0 -> 2
- net +12V: track 0.00 -> 14.0 mm
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- added copper zone on B.Cu, net GND
- added copper zone on F.Cu, net GND
Other:
- board size 47.5 x 97.7 mm -> 47 x 97.7 mm
